Commit message: change property names

File: semitrailer_description/urdf/semitrailer.urdf (robot description, URDF)
Before this commit: robot semitrailer, 6 links, 5 joints
Links:
- link tractor_link: geometry visual box size=${tractor_length} ${tractor_width} ${tractor_height}
- link trailer_link: geometry visual box size=${trailer_length} ${trailer_width} ${trailer_height}
Joints:
- joint coupler_joint: origin xyz=${trailer_width / 2} 0 0 -> xyz=${trailer_length / 2} 0 0
- joint tractor_joint: origin xyz=${hitch_length + tractor_width / 2} 0 0 -> xyz=${hitch_length + tractor_length / 2} 0 0
- joint tractor_steering_joint: origin xyz=${tractor_width / 2} 0 0 -> xyz=${tractor_length / 2} 0 0
- joint trailer_joint: origin xyz=${trailer_width / 2} 0 0 -> xyz=${trailer_length / 2} 0 0

Commit message: fix tractor steering description

File: semitrailer_description/urdf/semitrailer.urdf (robot description, URDF)
Before this commit: robot semitrailer, 6 links, 5 joints
Links:
- removed link tractor_steering_link
- added link tractor_steering_left_link
- added link tractor_steering_right_link
Joints:
- removed joint tractor_steering_joint
- added joint tractor_steering_left_joint: type continuous, parent tractor_link, child tractor_steering_left_link, origin xyz=${tractor_length / 2} ${tractor_width / 2} 0, axis 0 0 1
- added joint tractor_steering_right_joint: type continuous, parent tractor_link, child tractor_steering_right_link, origin xyz=${tractor_length / 2} ${-tractor_width / 2} 0, axis 0 0 1, mimic joint=tractor_steering_left_joint
